File: KiCad/AwesomeKeyboard_Left.kicad_pcb (KiCad board)
At the start: 2 copper layers, 140 x 109 mm, 57 parts, among them J1 AudioJack4_Ground, SW1 SW_DIP_x01, SW11 SW_Push, SW12 SW_Push, SW13 SW_Push, SW14 SW_Push, SW15 SW_Push, SW16 SW_Push, SW21 SW_Push, SW22 SW_Push, SW23 SW_Push, SW24 SW_Push, SW25 SW_Push, SW26 SW_Push, SW31 SW_Push, SW32 SW_Push, SW33 SW_Push, SW34 SW_Push, SW35 SW_Push, SW36 SW_Push, SW45 SW_Push, SW46 SW_Push

Commit message: modify
Parts:
- C1: footprint Capacitor_SMD:CP_Elec_3x5.3 -> Capacitor_THT:CP_Axial_L10.0mm_D4.5mm_P15.00mm_Horizontal
- D11, D12, D13, D14, D15, D16, D21, D22, D23, D24, D25, D26, D31, D32, D33, D34, D35, D36, D45, D46: footprint Diode_SMD:D_SOD-123 -> Diode_THT:D_DO-35_SOD27_P7.62mm_Horizontal
- LS1: footprint Buzzer_Beeper:Buzzer_Murata_PKMCS0909E4000-R1 -> Buzzer_Beeper:Buzzer_12x9.5RM7.6
- SW1: footprint Button_Switch_SMD:SW_DIP_SPSTx01_Slide_6.7x4.1mm_W6.73mm_P2.54mm_LowProfile_JPin -> Button_Switch_THT:SW_DIP_SPSTx01_Slide_6.7x4.1mm_W7.62mm_P2.54mm_LowProfile
- SW_RESET1: footprint Button_Switch_SMD:SW_SPST_FSMSM -> Button_Switch_THT:SW_PUSH_6mm
- moved D33 16.9 mm to (144.4, 137.3), turned to 90 degrees
- moved SW_RESET1 14.9 mm to (104.4, 167.0), turned to 180 degrees
- moved D23 11.6 mm to (140.3, 129.7)
- moved D13 11.5 mm to (141.4, 93.4)
- moved C1 11.1 mm to (132.6, 159.8), turned to 180 degrees
- moved D15 11.0 mm to (185.2, 98.1)
- moved D12 10.7 mm to (119.3, 104.9)
- moved D14 10.3 mm to (163.7, 98.6)
- moved D11 9.87 mm to (96.8, 115.7)
- moved R7 9.47 mm to (121.3, 154.1), turned to 0 degrees
- moved D25 9.46 mm to (184.4, 121.8)
- moved D21 9.46 mm to (96.4, 137.8)
- moved D35 9.44 mm to (184.4, 143.8)
- moved D22 9.24 mm to (118.2, 127.9)
- moved D24 9.15 mm to (162.1, 113.9)
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Connections:
- B1 pad 23: GND -> Net-(B1-Pad23)
Routing:
- net GND: track 349.4 -> 190.4 mm
- net Net-(B1-Pad22): track 62.1 -> 43.6 mm
- net /COL1: track 80.3 -> 63.4 mm
- net /COL2: track 67.1 -> 53.8 mm
- net Net-(R7-Pad1): track 22.3 -> 34.0 mm
- net /SPEAKER: track 49.8 -> 59.5 mm
- net Net-(D33-Pad1): track 11.7 -> 21.1 mm
- net /ROW3: track 441.8 -> 432.7 mm
- net /ROW2: track 276.7 -> 285.7 mm
- net Net-(D14-Pad1): track 16.7 -> 25.6 mm
- net Net-(D23-Pad1): track 17.5 -> 26.0 mm
- net /COL4: track 69.3 -> 60.8 mm
- net /COL3: track 75.8 -> 67.7 mm
- net VCC: track 176.5 -> 184.3 mm
- net /COL6: track 100.0 -> 92.6 mm
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