File: KiCad/_saved_AwesomeKeyboard_Left.sch (KiCad schematic (older format))
At the start: 57 parts, among them J1 AudioJack4_Ground, SW1 SW_DIP_x01, SW11 SW_Push, SW12 SW_Push, SW13 SW_Push, SW14 SW_Push, SW15 SW_Push, SW16 SW_Push, SW21 SW_Push, SW22 SW_Push, SW23 SW_Push, SW24 SW_Push, SW25 SW_Push, SW26 SW_Push, SW31 SW_Push, SW32 SW_Push, SW33 SW_Push, SW34 SW_Push, SW35 SW_Push, SW36 SW_Push, SW45 SW_Push, SW46 SW_Push

Commit message: modify
Parts:
- D11, D12, D13, D14, D15, D16, D21, D22, D23, D24, D25, D26, D31, D32, D33, D34, D35, D36, D45, D46: footprint Diode_THT:D_DO-35_SOD27_P10.16mm_Horizontal -> Diode_THT:D_DO-35_SOD27_P7.62mm_Horizontal
Connections:
- net GND: no longer B1.23 (GND)
- no-connect marks 2 -> 3
Changed lines of the file:
@@
 F 0 "D11" H 3900 2365 50  0000 C CNN
 F 1 "DIODE" H 3900 2274 50  0000 C CNN
-F 2 "Diode_THT:D_DO-35_SOD27_P10.16mm_Horizontal" H 3900 2100 50  0001 C CNN
+F 2 "Diode_THT:D_DO-35_SOD27_P7.62mm_Horizontal" H 3900 2100 50  0001 C CNN
 F 3 "~" H 3900 2100 50  0001 C CNN
 	1    3900 2100
@@
 F 0 "D16" H 7650 2365 50  0000 C CNN
 F 1 "DIODE" H 7650 2274 50  0000 C CNN
-F 2 "Diode_THT:D_DO-35_SOD27_P10.16mm_Horizontal" H 7650 2100 50  0001 C CNN
+F 2 "Diode_THT:D_DO-35_SOD27_P7.62mm_Horizontal" H 7650 2100 50  0001 C CNN
 F 3 "~" H 7650 2100 50  0001 C CNN
 	1    7650 2100
@@
 F 0 "D15" H 6900 2365 50  0000 C CNN
 F 1 "DIODE" H 6900 2274 50  0000 C CNN
-F 2 "Diode_THT:D_DO-35_SOD27_P10.16mm_Horizontal" H 6900 2100 50  0001 C CNN
+F 2 "Diode_THT:D_DO-35_SOD27_P7.62mm_Horizontal" H 6900 2100 50  0001 C CNN
 F 3 "~" H 6900 2100 50  0001 C CNN
 	1    6900 2100
@@
 F 0 "D14" H 6150 2365 50  0000 C CNN
 F 1 "DIODE" H 6150 2274 50  0000 C CNN
-F 2 "Diode_THT:D_DO-35_SOD27_P10.16mm_Horizontal" H 6150 2100 50  0001 C CNN
+F 2 "Diode_THT:D_DO-35_SOD27_P7.62mm_Horizontal" H 6150 2100 50  0001 C CNN
 F 3 "~" H 6150 2100 50  0001 C CNN
 	1    6150 2100
@@
 F 0 "D13" H 5400 2365 50  0000 C CNN
 F 1 "DIODE" H 5400 2274 50  0000 C CNN
-F 2 "Diode_THT:D_DO-35_SOD27_P10.16mm_Horizontal" H 5400 2100 50  0001 C CNN
+F 2 "Diode_THT:D_DO-35_SOD27_P7.62mm_Horizontal" H 5400 2100 50  0001 C CNN
 F 3 "~" H 5400 2100 50  0001 C CNN
 	1    5400 2100
@@
 F 0 "D12" H 4650 2365 50  0000 C CNN
 F 1 "DIODE" H 4650 2274 50  0000 C CNN
-F 2 "Diode_THT:D_DO-35_SOD27_P10.16mm_Horizontal" H 4650 2100 50  0001 C CNN
+F 2 "Diode_THT:D_DO-35_SOD27_P7.62mm_Horizontal" H 4650 2100 50  0001 C CNN
 F 3 "~" H 4650 2100 50  0001 C CNN
 	1    4650 2100
@@
 F 0 "D36" H 7650 3765 50  0000 C CNN
 F 1 "DIODE" H 7650 3674 50  0000 C CNN
-F 2 "Diode_THT:D_DO-35_SOD27_P10.16mm_Horizontal" H 7650 3500 50  0001 C CNN
+F 2 "Diode_THT:D_DO-35_SOD27_P7.62mm_Horizontal" H 7650 3500 50  0001 C CNN
 F 3 "~" H 7650 3500 50  0001 C CNN
 	1    7650 3500
@@
 F 0 "D35" H 6900 3765 50  0000 C CNN
 F 1 "DIODE" H 6900 3674 50  0000 C CNN
-F 2 "Diode_THT:D_DO-35_SOD27_P10.16mm_Horizontal" H 6900 3500 50  0001 C CNN
+F 2 "Diode_THT:D_DO-35_SOD27_P7.62mm_Horizontal" H 6900 3500 50  0001 C CNN
 F 3 "~" H 6900 3500 50  0001 C CNN
 	1    6900 3500
@@
 F 0 "D26" H 7650 3065 50  0000 C CNN
 F 1 "DIODE" H 7650 2974 50  0000 C CNN
-F 2 "Diode_THT:D_DO-35_SOD27_P10.16mm_Horizontal" H 7650 2800 50  0001 C CNN
+F 2 "Diode_THT:D_DO-35_SOD27_P7.62mm_Horizontal" H 7650 2800 50  0001 C CNN
 F 3 "~" H 7650 2800 50  0001 C CNN
 	1    7650 2800
@@
 F 0 "D25" H 6900 3065 50  0000 C CNN
 F 1 "DIODE" H 6900 2974 50  0000 C CNN
-F 2 "Diode_THT:D_DO-35_SOD27_P10.16mm_Horizontal" H 6900 2800 50  0001 C CNN
+F 2 "Diode_THT:D_DO-35_SOD27_P7.62mm_Horizontal" H 6900 2800 50  0001 C CNN
 F 3 "~" H 6900 2800 50  0001 C CNN
 	1    6900 2800
@@
 F 0 "D34" H 6150 3765 50  0000 C CNN
 F 1 "DIODE" H 6150 3674 50  0000 C CNN
-F 2 "Diode_THT:D_DO-35_SOD27_P10.16mm_Horizontal" H 6150 3500 50  0001 C CNN
+F 2 "Diode_THT:D_DO-35_SOD27_P7.62mm_Horizontal" H 6150 3500 50  0001 C CNN
 F 3 "~" H 6150 3500 50  0001 C CNN
 	1    6150 3500
@@
 F 0 "D33" H 5400 3765 50  0000 C CNN
 F 1 "DIODE" H 5400 3674 50  0000 C CNN
-F 2 "Diode_THT:D_DO-35_SOD27_P10.16mm_Horizontal" H 5400 3500 50  0001 C CNN
+F 2 "Diode_THT:D_DO-35_SOD27_P7.62mm_Horizontal" H 5400 3500 50  0001 C CNN
 F 3 "~" H 5400 3500 50  0001 C CNN
 	1    5400 3500
@@
 F 0 "D24" H 6150 3065 50  0000 C CNN
 F 1 "DIODE" H 6150 2974 50  0000 C CNN
-F 2 "Diode_THT:D_DO-35_SOD27_P10.16mm_Horizontal" H 6150 2800 50  0001 C CNN
+F 2 "Diode_THT:D_DO-35_SOD27_P7.62mm_Horizontal" H 6150 2800 50  0001 C CNN
 F 3 "~" H 6150 2800 50  0001 C CNN
 	1    6150 2800
@@
 F 0 "D23" H 5400 3065 50  0000 C CNN
 F 1 "DIODE" H 5400 2974 50  0000 C CNN
-F 2 "Diode_THT:D_DO-35_SOD27_P10.16mm_Horizontal" H 5400 2800 50  0001 C CNN
+F 2 "Diode_THT:D_DO-35_SOD27_P7.62mm_Horizontal" H 5400 2800 50  0001 C CNN
 F 3 "~" H 5400 2800 50  0001 C CNN
 	1    5400 2800
@@
 F 0 "D46" H 7650 4465 50  0000 C CNN
 F 1 "DIODE" H 7650 4374 50  0000 C CNN
-F 2 "Diode_THT:D_DO-35_SOD27_P10.16mm_Horizontal" H 7650 4200 50  0001 C CNN
+F 2 "Diode_THT:D_DO-35_SOD27_P7.62mm_Horizontal" H 7650 4200 50  0001 C CNN
 F 3 "~" H 7650 4200 50  0001 C CNN
 	1    7650 4200
@@
 F 0 "D45" H 6900 4465 50  0000 C CNN
 F 1 "DIODE" H 6900 4374 50  0000 C CNN
-F 2 "Diode_THT:D_DO-35_SOD27_P10.16mm_Horizontal" H 6900 4200 50  0001 C CNN
+F 2 "Diode_THT:D_DO-35_SOD27_P7.62mm_Horizontal" H 6900 4200 50  0001 C CNN
 F 3 "~" H 6900 4200 50  0001 C CNN
 	1    6900 4200
@@
 F 0 "D32" H 4650 3765 50  0000 C CNN
 F 1 "DIODE" H 4650 3674 50  0000 C CNN
-F 2 "Diode_THT:D_DO-35_SOD27_P10.16mm_Horizontal" H 4650 3500 50  0001 C CNN
+F 2 "Diode_THT:D_DO-35_SOD27_P7.62mm_Horizontal" H 4650 3500 50  0001 C CNN
 F 3 "~" H 4650 3500 50  0001 C CNN
 	1    4650 3500
@@
 F 0 "D31" H 3900 3765 50  0000 C CNN
 F 1 "DIODE" H 3900 3674 50  0000 C CNN
-F 2 "Diode_THT:D_DO-35_SOD27_P10.16mm_Horizontal" H 3900 3500 50  0001 C CNN
+F 2 "Diode_THT:D_DO-35_SOD27_P7.62mm_Horizontal" H 3900 3500 50  0001 C CNN
 F 3 "~" H 3900 3500 50  0001 C CNN
 	1    3900 3500
@@
 F 0 "D22" H 4650 3065 50  0000 C CNN
 F 1 "DIODE" H 4650 2974 50  0000 C CNN
-F 2 "Diode_THT:D_DO-35_SOD27_P10.16mm_Horizontal" H 4650 2800 50  0001 C CNN
+F 2 "Diode_THT:D_DO-35_SOD27_P7.62mm_Horizontal" H 4650 2800 50  0001 C CNN
 F 3 "~" H 4650 2800 50  0001 C CNN
 	1    4650 2800
@@
 F 0 "D21" H 3900 3065 50  0000 C CNN
 F 1 "DIODE" H 3900 2974 50  0000 C CNN
-F 2 "Diode_THT:D_DO-35_SOD27_P10.16mm_Horizontal" H 3900 2800 50  0001 C CNN
+F 2 "Diode_THT:D_DO-35_SOD27_P7.62mm_Horizontal" H 3900 2800 50  0001 C CNN
 F 3 "~" H 3900 2800 50  0001 C CNN
 	1    3900 2800
@@
 	4550 7100 4550 7200
 Wire Wire Line
-	4350 6600 4350 6650
-Wire Wire Line
 	4650 6850 4650 6650
 $Comp
@@
 Wire Wire Line
 	4650 6650 4650 6550
-Connection ~ 4350 6650
 Wire Wire Line
 	4350 6650 4350 7200
@@
 Wire Wire Line
 	4350 7200 4550 7200
-Wire Wire Line
-	4350 6600 4450 6600
-Wire Wire Line
-	4450 6600 4450 6550
+NoConn ~ 4450 6550
 $EndSCHEMATC
