File: KiCad_right/AwesomeKeyboard_Right.sch (KiCad schematic (older format))
At the start: 57 parts, among them J1 AudioJack4_Ground, SW1 SW_DIP_x01, SW11 SW_Push, SW12 SW_Push, SW13 SW_Push, SW14 SW_Push, SW15 SW_Push, SW16 SW_Push, SW21 SW_Push, SW22 SW_Push, SW23 SW_Push, SW24 SW_Push, SW25 SW_Push, SW26 SW_Push, SW31 SW_Push, SW32 SW_Push, SW33 SW_Push, SW34 SW_Push, SW35 SW_Push, SW36 SW_Push, SW45 SW_Push, SW46 SW_Push

Commit message: a
Parts:
- removed C1: C, Capacitor_THT:CP_Axial_L10.0mm_D4.5mm_P15.00mm_Horizontal, symbol Device:C
- removed R1, R2: R, Resistor_THT:R_Axial_DIN0204_L3.6mm_D1.6mm_P7.62mm_Horizontal, symbol Device:R
- J1: symbol AwesomeKeyboard_Left-rescue:AudioJack4_Ground-my_trrs -> AwesomeKeyboard_Right-rescue:AudioJack4_Ground-my_trrs-AwesomeKeyboard_Left-rescue
Connections:
- wire segments 95 -> 83
- no-connect marks 2 -> 5
Other:
- moved on the sheet: B1, D11, D12, D13, D14, D15, D16, D21, D22, D23, D24, D25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

Commit message: right
Connections:
- net GND: now also B1.3 (GND), B1.4 (GND)
- net VCC: now also B1.21 (VCC)
- no-connect marks 5 -> 1
Changed lines of the file:
@@
 Text Label 9350 4700 2    50   ~ 0
 COL6
-NoConn ~ 9050 4000
 Wire Wire Line
 	8150 4100 7850 4100
@@
 Wire Wire Line
 	9300 3800 9650 3800
-NoConn ~ 9050 3900
-NoConn ~ 8150 3800
-NoConn ~ 8150 4000
+$Comp
+L power:VCC #PWR0104
+U 1 1 5C269825
+P 8150 4000
+F 0 "#PWR0104" H 8150 3850 50  0001 C CNN
+F 1 "VCC" V 8168 4127 50  0000 L CNN
+F 2 "" H 8150 4000 50  0001 C CNN
+F 3 "" H 8150 4000 50  0001 C CNN
+	1    8150 4000
+	0    -1   -1   0
+$EndComp
+$Comp
+L power:GND #PWR0105
+U 1 1 5C26996A
+P 9050 3900
+F 0 "#PWR0105" H 9050 3650 50  0001 C CNN
+F 1 "GND" V 9055 3772 50  0000 R CNN
+F 2 "" H 9050 3900 50  0001 C CNN
+F 3 "" H 9050 3900 50  0001 C CNN
+	1    9050 3900
+	0    -1   -1   0
+$EndComp
+$Comp
+L power:GND #PWR0113
+U 1 1 5C269A9A
+P 9050 4000
+F 0 "#PWR0113" H 9050 3750 50  0001 C CNN
+F 1 "GND" V 9055 3872 50  0000 R CNN
+F 2 "" H 9050 4000 50  0001 C CNN
+F 3 "" H 9050 4000 50  0001 C CNN
+	1    9050 4000
+	0    -1   -1   0
+$EndComp
 $EndSCHEMATC

Commit message: left
Connections:
- net COL1: now also B1.19 (A2); no longer B1.1 (TXO)
- net COL2: now also B1.18 (A1); no longer B1.2 (RXI)
- net COL3: now also B1.17 (A0); no longer B1.8 (*5)
- net COL4: now also B1.16 (13(SCK)); no longer B1.9 (*6)
- net COL5: now also B1.15 (12(MISO)); no longer B1.10 (7)
- net COL6: now also B1.14 (11(MOSI)); no longer B1.11 (8)
- net GND: now also B1.23 (GND)
- net LED1: now also B1.12 (*9); no longer B1.13 (*10)
- net LED2: now also B1.11 (8); no longer B1.14 (11(MOSI))
- net LED3: now also B1.10 (7); no longer B1.15 (12(MISO))
- net LED4: now also B1.9 (*6); no longer B1.16 (13(SCK))
- net ROW1: now also B1.8 (*5), SW11.1, SW12.1, SW13.1, SW14.1, SW15.1, SW16.1; no longer B1.17 (A0), SW11.2, SW12.2, SW13.2, SW14.2, SW15.2, SW16.2
- net ROW2: now also B1.7 (4), SW21.1, SW22.1, SW23.1, SW24.1, SW25.1, SW26.1; no longer B1.18 (A1), SW21.2, SW22.2, SW23.2, SW24.2, SW25.2, SW26.2
- net ROW3: now also B1.2 (RXI), SW31.1, SW32.1, SW33.1, SW34.1, SW35.1, SW36.1; no longer B1.19 (A2), SW31.2, SW32.2, SW33.2, SW34.2, SW35.2, SW36.2
- net ROW4: now also B1.13 (*10), SW45.1, SW46.1; no longer B1.12 (*9), SW45.2, SW46.2
- net SPEAKER: now also B1.1 (TXO); no longer B1.20 (A3)
- net at D11.1 (K): now also SW11.2; no longer SW11.1
- net at D12.1 (K): now also SW12.2; no longer SW12.1
- net at D21.1 (K): now also SW21.2; no longer SW21.1
- net at D22.1 (K): now also SW22.2; no longer SW22.1
- net at D31.1 (K): now also SW31.2; no longer SW31.1
- net at D32.1 (K): now also SW32.2; no longer SW32.1
- net at D45.1 (K): now also SW45.2; no longer SW45.1
- net at D46.1 (K): now also SW46.2; no longer SW46.1
- net at D13.1 (K): now also SW13.2; no longer SW13.1
- net at D14.1 (K): now also SW14.2; no longer SW14.1
- net at D23.1 (K): now also SW23.2; no longer SW23.1
- net at D24.1 (K): now also SW24.2; no longer SW24.1
- net at D33.1 (K): now also SW33.2; no longer SW33.1
- net at D34.1 (K): now also SW34.2; no longer SW34.1
- net at D15.1 (K): now also SW15.2; no longer SW15.1
- net at D16.1 (K): now also SW16.2; no longer SW16.1
- net at D25.1 (K): now also SW25.2; no longer SW25.1
- net at D26.1 (K): now also SW26.2; no longer SW26.1
- net at D35.1 (K): now also SW35.2; no longer SW35.1
- net at D36.1 (K): now also SW36.2; no longer SW36.1
- no-connect marks 1 -> 0
Other:
- moved on the sheet: J1, SW_RESET1
Changed lines of the file:
@@
 F 3 "" H 6350 2300 50  0001 C CNN
 	1    6350 2100
-	0    1    -1   0
+	0    1    1    0
 $EndComp
 $Comp
@@
 F 3 "" H 2600 2300 50  0001 C CNN
 	1    2600 2100
-	0    1    -1   0
+	0    1    1    0
 $EndComp
 $Comp
@@
 F 3 "" H 3350 2300 50  0001 C CNN
 	1    3350 2100
-	0    1    -1   0
+	0    1    1    0
 $EndComp
 $Comp
@@
 F 3 "" H 4100 2300 50  0001 C CNN
 	1    4100 2100
-	0    1    -1   0
+	0    1    1    0
 $EndComp
 $Comp
@@
 F 3 "" H 4850 2300 50  0001 C CNN
 	1    4850 2100
-	0    1    -1   0
+	0    1    1    0
 $EndComp
 $Comp
@@
 F 3 "" H 5600 2300 50  0001 C CNN
 	1    5600 2100
-	0    1    -1   0
+	0    1    1    0
 $EndComp
 $Comp
@@
 F 3 "" H 2600 3700 50  0001 C CNN
 	1    2600 3500
-	0    1    -1   0
+	0    1    1    0
 $EndComp
 $Comp
@@
 F 3 "" H 3350 3700 50  0001 C CNN
 	1    3350 3500
-	0    1    -1   0
+	0    1    1    0
 $EndComp
 $Comp
@@
 F 3 "" H 2600 3000 50  0001 C CNN
 	1    2600 2800
-	0    1    -1   0
+	0    1    1    0
 $EndComp
 $Comp
@@
 F 3 "" H 3350 3000 50  0001 C CNN
 	1    3350 2800
-	0    1    -1   0
+	0    1    1    0
 $EndComp
 $Comp
@@
 F 3 "" H 4100 3700 50  0001 C CNN
 	1    4100 3500
-	0    1    -1   0
+	0    1    1    0
 $EndComp
 $Comp
@@
 F 3 "" H 4850 3700 50  0001 C CNN
 	1    4850 3500
-	0    1    -1   0
+	0    1    1    0
 $EndComp
 $Comp
@@
 F 3 "" H 4100 3000 50  0001 C CNN
 	1    4100 2800
-	0    1    -1   0
+	0    1    1    0
 $EndComp
 $Comp
@@
 F 3 "" H 4850 3000 50  0001 C CNN
 	1    4850 2800
-	0    1    -1   0
+	0    1    1    0
 $EndComp
 $Comp
@@
 F 3 "" H 2600 4400 50  0001 C CNN
 	1    2600 4200
-	0    1    -1   0
+	0    1    1    0
 $EndComp
 $Comp
@@
 F 3 "" H 3350 4400 50  0001 C CNN
 	1    3350 4200
-	0    1    -1   0
+	0    1    1    0
 $EndComp
 $Comp
@@
 F 3 "" H 5600 3700 50  0001 C CNN
 	1    5600 3500
-	0    1    -1   0
+	0    1    1    0
 $EndComp
 $Comp
@@
 F 3 "" H 6350 3700 50  0001 C CNN
 	1    6350 3500
-	0    1    -1   0
+	0    1    1    0
 $EndComp
 $Comp
@@
 F 3 "" H 5600 3000 50  0001 C CNN
 	1    5600 2800
-	0    1    -1   0
+	0    1    1    0
 $EndComp
 $Comp
@@
 F 3 "" H 6350 3000 50  0001 C CNN
 	1    6350 2800
-	0    1    -1   0
+	0    1    1    0
 $EndComp
 $Comp
@@
 Text Label 7850 4300 0    50   ~ 0
 ROW2
-Text Label 7850 4200 0    50   ~ 0
+Text Label 7850 3800 0    50   ~ 0
 ROW3
 Wire Wire Line
@@
 Wire Wire Line
 	8150 4300 7850 4300
-Wire Wire Line
-	8150 4200 7850 4200
 Wire Wire Line
 	8150 4700 7850 4700
@@
 ROW4
 Wire Wire Line
-	9650 4300 9650 4450
+	7550 4300 7550 4450
 $Comp
 L power:GND #PWR0101
 U 1 1 5BF85540
-P 9650 4450
-F 0 "#PWR0101" H 9650 4200 50  0001 C CNN
-F 1 "GND" H 9655 4277 50  0000 C CNN
-F 2 "" H 9650 4450 50  0001 C CNN
-F 3 "" H 9650 4450 50  0001 C CNN
-	1    9650 4450
+P 7550 4450
+F 0 "#PWR0101" H 7550 4200 50  0001 C CNN
+F 1 "GND" H 7555 4277 50  0000 C CNN
+F 2 "" H 7550 4450 50  0001 C CNN
+F 3 "" H 7550 4450 50  0001 C CNN
+	1    7550 4450
 	-1   0    0    -1
 $EndComp
@@
 L power:VCC #PWR0102
 U 1 1 5BF855E7
-P 9300 3650
-F 0 "#PWR0102" H 9300 3500 50  0001 C CNN
-F 1 "VCC" H 9317 3823 50  0000 C CNN
-F 2 "" H 9300 3650 50  0001 C CNN
-F 3 "" H 9300 3650 50  0001 C CNN
-	1    9300 3650
-	-1   0    0    -1
-$EndComp
-Text Label 7850 4100 0    50   ~ 0
+P 7550 3650
+F 0 "#PWR0102" H 7550 3500 50  0001 C CNN
+F 1 "VCC" H 7567 3823 50  0000 C CNN
+F 2 "" H 7550 3650 50  0001 C CNN
+F 3 "" H 7550 3650 50  0001 C CNN
+	1    7550 3650
+	-1   0    0    -1
+$EndComp
+Text Label 7850 3700 0    50   ~ 0
 SPEAKER
 $Comp
 L Switch:SW_Push SW_RESET1
 U 1 1 5BF8FEF5
-P 7800 3900
-F 0 "SW_RESET1" H 7800 4185 50  0000 C CNN
-F 1 "SW_Push" H 7800 4094 50  0000 C CNN
-F 2 "Button_Switch_THT:SW_PUSH_6mm" H 7800 4100 50  0001 C CNN
-F 3 "" H 7800 4100 50  0001 C CNN
-	1    7800 3900
-	-1   0    0    -1
+P 9400 3900
+F 0 "SW_RESET1" H 9400 4185 50  0000 C CNN
+F 1 "SW_Push" H 9400 4094 50  0000 C CNN
+F 2 "Button_Switch_THT:SW_PUSH_6mm" H 9400 4100 50  0001 C CNN
+F 3 "" H 9400 4100 50  0001 C CNN
+	1    9400 3900
+	1    0    0    -1
 $EndComp
 $Comp
@@
 Wire Wire Line
 	2250 6050 2250 6150
-Wire Wire Line
-	9650 4000 9650 3800
-Wire Wire Line
-	9300 3800 9300 3650
 $Comp
 L AwesomeKeyboard_Right-rescue:AudioJack4_Ground-my_trrs-AwesomeKeyboard_Left-rescue J1
 U 1 1 5C055710
-P 9850 4100
-F 0 "J1" H 9816 4442 50  0000 C CNN
-F 1 "AudioJack4_Ground" H 9816 4351 50  0000 C CNN
-F 2 "Connector_Audio:Jack_3.5mm_PJ320D_Horizontal" H 9850 4100 50  0001 C CNN
-F 3 "" H 9850 4100 50  0001 C CNN
-	1    9850 4100
-	-1   0    0    -1
+P 7350 4100
+F 0 "J1" H 7316 4442 50  0000 C CNN
+F 1 "AudioJack4_Ground" H 7316 4351 50  0000 C CNN
+F 2 "Connector_Audio:Jack_3.5mm_PJ320D_Horizontal" H 7350 4100 50  0001 C CNN
+F 3 "" H 7350 4100 50  0001 C CNN
+	1    7350 4100
+	1    0    0    -1
 $EndComp
 Connection ~ 2950 3700
@@
 Text Label 7850 4500 0    50   ~ 0
 LED4
-Text Label 9150 3450 1    50   ~ 0
+Text Label 9300 4300 0    50   ~ 0
 COL2
-Text Label 9050 3450 1    50   ~ 0
+Text Label 9300 4200 0    50   ~ 0
 COL1
 $Comp
@@
 	3000 5950 3450 5950
 Wire Wire Line
-	9050 3700 9050 3450
-Wire Wire Line
-	9050 3800 9150 3800
-Wire Wire Line
-	9150 3800 9150 3450
+	9050 4200 9300 4200
 $Comp
 L SparkFun-Boards:SPARKFUN_PRO_MICRO B1
@@
 F 4 "000-00000" H 8600 4981 60  0000 C CNN "フィールド4"
 	1    8600 4250
-	-1   0    0    -1
+	1    0    0    -1
 $EndComp
 Wire Wire Line
@@
 $EndComp
 Wire Wire Line
-	7600 3900 7500 3900
+	9600 3900 9700 3900
 $Comp
 L power:GND #PWR0103
 U 1 1 5BF8AB0F
-P 7500 3900
-F 0 "#PWR0103" H 7500 3650 50  0001 C CNN
-F 1 "GND" H 7505 3727 50  0000 C CNN
-F 2 "" H 7500 3900 50  0001 C CNN
-F 3 "" H 7500 3900 50  0001 C CNN
-	1    7500 3900
-	-1   0    0    -1
+P 9700 3900
+F 0 "#PWR0103" H 9700 3650 50  0001 C CNN
+F 1 "GND" H 9705 3727 50  0000 C CNN
+F 2 "" H 9700 3900 50  0001 C CNN
+F 3 "" H 9700 3900 50  0001 C CNN
+	1    9700 3900
+	1    0    0    -1
 $EndComp
 $Comp
@@
 COL6
 Wire Wire Line
-	8150 4100 7850 4100
-NoConn ~ 8150 3700
-Wire Wire Line
-	8150 3900 8000 3900
-Wire Wire Line
-	9050 4100 9650 4100
-Wire Wire Line
-	9050 4200 9650 4200
-Wire Wire Line
-	9300 3800 9650 3800
+	8150 3700 7850 3700
+Wire Wire Line
+	9050 3900 9200 3900
+Wire Wire Line
+	8150 4100 7550 4100
+Wire Wire Line
+	8150 4200 7550 4200
 $Comp
 L power:VCC #PWR0104
 U 1 1 5C269825
+P 9050 4000
+F 0 "#PWR0104" H 9050 3850 50  0001 C CNN
+F 1 "VCC" V 9068 4127 50  0000 L CNN
+F 2 "" H 9050 4000 50  0001 C CNN
+F 3 "" H 9050 4000 50  0001 C CNN
+	1    9050 4000
+	0    1    -1   0
+$EndComp
+$Comp
+L power:GND #PWR0105
+U 1 1 5C26996A
+P 8150 3900
+F 0 "#PWR0105" H 8150 3650 50  0001 C CNN
+F 1 "GND" V 8155 3772 50  0000 R CNN
+F 2 "" H 8150 3900 50  0001 C CNN
+F 3 "" H 8150 3900 50  0001 C CNN
+	1    8150 3900
+	0    1    -1   0
+$EndComp
+$Comp
+L power:GND #PWR0113
+U 1 1 5C269A9A
+P 9050 3800
+F 0 "#PWR0113" H 9050 3550 50  0001 C CNN
+F 1 "GND" V 9055 3672 50  0000 R CNN
+F 2 "" H 9050 3800 50  0001 C CNN
+F 3 "" H 9050 3800 50  0001 C CNN
+	1    9050 3800
+	0    -1   -1   0
+$EndComp
+$Comp
+L power:GND #PWR0114
+U 1 1 5C2B6ACD
 P 8150 4000
-F 0 "#PWR0104" H 8150 3850 50  0001 C CNN
-F 1 "VCC" V 8168 4127 50  0000 L CNN
+F 0 "#PWR0114" H 8150 3750 50  0001 C CNN
+F 1 "GND" V 8155 3872 50  0000 R CNN
 F 2 "" H 8150 4000 50  0001 C CNN
 F 3 "" H 8150 4000 50  0001 C CNN
 	1    8150 4000
-	0    -1   -1   0
-$EndComp
-$Comp
-L power:GND #PWR0105
-U 1 1 5C26996A
-P 9050 3900
-F 0 "#PWR0105" H 9050 3650 50  0001 C CNN
-F 1 "GND" V 9055 3772 50  0000 R CNN
-F 2 "" H 9050 3900 50  0001 C CNN
-F 3 "" H 9050 3900 50  0001 C CNN
-	1    9050 3900
-	0    -1   -1   0
-$EndComp
-$Comp
-L power:GND #PWR0113
-U 1 1 5C269A9A
-P 9050 4000
-F 0 "#PWR0113" H 9050 3750 50  0001 C CNN
-F 1 "GND" V 9055 3872 50  0000 R CNN
-F 2 "" H 9050 4000 50  0001 C CNN
-F 3 "" H 9050 4000 50  0001 C CNN
-	1    9050 4000
-	0    -1   -1   0
-$EndComp
+	0    1    -1   0
+$EndComp
+Wire Wire Line
+	7550 3650 7550 4000
+Wire Wire Line
+	7850 3800 8150 3800
+Wire Wire Line
+	9050 4300 9300 4300
 $EndSCHEMATC

Commit message: right
Connections:
- net LED1: now also B1.11 (8); no longer B1.12 (*9)
- net LED2: now also B1.10 (7); no longer B1.11 (8)
- net LED3: now also B1.9 (*6); no longer B1.10 (7)
- net LED4: now also B1.8 (*5); no longer B1.9 (*6)
- net ROW1: now also B1.12 (*9); no longer B1.8 (*5)
Changed lines of the file:
@@
 Wire Wire Line
 	9050 4700 9350 4700
-Text Label 7850 4400 0    50   ~ 0
+Text Label 7850 4800 0    50   ~ 0
 ROW1
 Text Label 7850 4300 0    50   ~ 0
@@
 ROW3
 Wire Wire Line
-	8150 4400 7850 4400
+	8150 4800 7850 4800
 Wire Wire Line
 	8150 4300 7850 4300
 Wire Wire Line
-	8150 4700 7850 4700
+	8150 4600 7850 4600
+Text Label 7850 4600 0    50   ~ 0
+LED2
 Text Label 7850 4700 0    50   ~ 0
-LED2
-Text Label 7850 4800 0    50   ~ 0
 LED1
 Text Label 9350 4400 2    50   ~ 0
@@
 ROW4
 Wire Wire Line
-	8150 4800 7850 4800
+	8150 4700 7850 4700
 Wire Wire Line
 	9350 4400 9050 4400
@@
 $EndComp
 Wire Wire Line
-	8150 4600 7850 4600
-Wire Wire Line
 	8150 4500 7850 4500
-Text Label 7850 4600 0    50   ~ 0
+Wire Wire Line
+	8150 4400 7850 4400
+Text Label 7850 4500 0    50   ~ 0
 LED3
-Text Label 7850 4500 0    50   ~ 0
+Text Label 7850 4400 0    50   ~ 0
 LED4
 Text Label 9300 4300 0    50   ~ 0

Commit message: re
Parts:
- removed J1: AudioJack4_Ground, Connector_Audio:Jack_3.5mm_PJ320D_Horizontal, symbol AwesomeKeyboard_Right-rescue:AudioJack4_Ground-my_trrs-AwesomeKeyboard_Left-res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
- removed LED3, LED4: LED, LED_THT:LED_D5.0mm, symbol Device:LED
- removed R5, R6: R, Resistor_THT:R_Axial_DIN0204_L3.6mm_D1.6mm_P7.62mm_Horizontal, symbol Device:R
- added J_joystick1, J_trrs1: 4P4C, Connector_PinHeader_2.00mm:PinHeader_1x04_P2.00mm_Vertical, symbol Connector:4P4C
Connections:
- net LED3 is gone; now on net LED1: B1.9 (*6)
- net LED4 is gone; now on net LED2: B1.8 (*5)
- net GND: now also J_joystick1.1, J_trrs1.3
- net LED1: no longer B1.11 (8)
- net LED2: no longer B1.10 (7)
- net ROW1: now also B1.20 (A3); no longer B1.12 (*9)
- net VCC: now also J_joystick1.4, J_trrs1.4
- net at B1.5 (2): now also J_trrs1.2
- net at B1.6 (*3): now also J_trrs1.1
- new net X1: B1.10 (7), J_joystick1.2
- new net Y1: B1.11 (8), J_joystick1.3
Changed lines of the file:
@@
 Wire Wire Line
 	9050 4700 9350 4700
-Text Label 7850 4800 0    50   ~ 0
+Text Label 9350 4100 2    50   ~ 0
 ROW1
 Text Label 7850 4300 0    50   ~ 0
@@
 ROW3
 Wire Wire Line
-	8150 4800 7850 4800
+	9050 4100 9350 4100
 Wire Wire Line
 	8150 4300 7850 4300
 Wire Wire Line
-	8150 4600 7850 4600
+	8150 4700 7850 4700
+Text Label 7850 4700 0    50   ~ 0
+Y1
 Text Label 7850 4600 0    50   ~ 0
-LED2
-Text Label 7850 4700 0    50   ~ 0
-LED1
+X1
 Text Label 9350 4400 2    50   ~ 0
 COL3
@@
 ROW4
 Wire Wire Line
-	8150 4700 7850 4700
+	8150 4600 7850 4600
 Wire Wire Line
 	9350 4400 9050 4400
@@
 Text Label 3850 4000 2    50   ~ 0
 ROW4
-Wire Wire Line
-	7550 4300 7550 4450
-$Comp
-L power:GND #PWR0101
-U 1 1 5BF85540
-P 7550 4450
-F 0 "#PWR0101" H 7550 4200 50  0001 C CNN
-F 1 "GND" H 7555 4277 50  0000 C CNN
-F 2 "" H 7550 4450 50  0001 C CNN
-F 3 "" H 7550 4450 50  0001 C CNN
-	1    7550 4450
-	-1   0    0    -1
-$EndComp
-$Comp
-L power:VCC #PWR0102
-U 1 1 5BF855E7
-P 7550 3650
-F 0 "#PWR0102" H 7550 3500 50  0001 C CNN
-F 1 "VCC" H 7567 3823 50  0000 C CNN
-F 2 "" H 7550 3650 50  0001 C CNN
-F 3 "" H 7550 3650 50  0001 C CNN
-	1    7550 3650
-	-1   0    0    -1
-$EndComp
 Text Label 7850 3700 0    50   ~ 0
 SPEAKER
@@
 Wire Wire Line
 	2250 6050 2250 6150
-$Comp
-L AwesomeKeyboard_Right-rescue:AudioJack4_Ground-my_trrs-AwesomeKeyboard_Left-rescue J1
-U 1 1 5C055710
-P 7350 4100
-F 0 "J1" H 7316 4442 50  0000 C CNN
-F 1 "AudioJack4_Ground" H 7316 4351 50  0000 C CNN
-F 2 "Connector_Audio:Jack_3.5mm_PJ320D_Horizontal" H 7350 4100 50  0001 C CNN
-F 3 "" H 7350 4100 50  0001 C CNN
-	1    7350 4100
-	1    0    0    -1
-$EndComp
 Connection ~ 2950 3700
 Connection ~ 2200 3700
@@
 	8150 4400 7850 4400
 Text Label 7850 4500 0    50   ~ 0
-LED3
+LED1
 Text Label 7850 4400 0    50   ~ 0
-LED4
+LED2
 Text Label 9300 4300 0    50   ~ 0
 COL2
@@
 	-1   0    0    -1
 $EndComp
-$Comp
-L Device:LED LED3
-U 1 1 5C089824
-P 9850 1400
-F 0 "LED3" H 9842 1616 50  0000 C CNN
-F 1 "LED" H 9842 1525 50  0000 C CNN
-F 2 "LED_THT:LED_D5.0mm" H 9850 1400 50  0001 C CNN
-F 3 "~" H 9850 1400 50  0001 C CNN
-	1    9850 1400
-	-1   0    0    -1
-$EndComp
-$Comp
-L Device:LED LED4
-U 1 1 5C08982B
-P 10350 1400
-F 0 "LED4" H 10342 1616 50  0000 C CNN
-F 1 "LED" H 10342 1525 50  0000 C CNN
-F 2 "LED_THT:LED_D5.0mm" H 10350 1400 50  0001 C CNN
-F 3 "~" H 10350 1400 50  0001 C CNN
-	1    10350 1400
-	-1   0    0    -1
-$EndComp
 Wire Wire Line
 	8700 1750 8700 2050
@@
 Wire Wire Line
 	9500 1400 9500 1700
-Wire Wire Line
-	9700 1750 9700 2050
-Wire Wire Line
-	10000 1400 10000 1700
-Wire Wire Line
-	10200 1750 10200 2050
-Wire Wire Line
-	10500 1400 10500 1700
 Text Label 8700 2050 0    50   ~ 0
 LED1
 Text Label 9200 2050 0    50   ~ 0
 LED2
-Text Label 9700 2050 0    50   ~ 0
-LED3
-Text Label 10200 2050 0    50   ~ 0
-LED4
 $Comp
 L power:GND #PWR0109
@@
 $EndComp
 $Comp
-L power:GND #PWR0111
-U 1 1 5C0A1730
-P 10000 1700
-F 0 "#PWR0111" H 10000 1450 50  0001 C CNN
-F 1 "GND" H 10005 1527 50  0000 C CNN
-F 2 "" H 10000 1700 50  0001 C CNN
-F 3 "" H 10000 1700 50  0001 C CNN
-	1    10000 1700
-	1    0    0    -1
-$EndComp
-$Comp
-L power:GND #PWR0112
-U 1 1 5C0A17B6
-P 10500 1700
-F 0 "#PWR0112" H 10500 1450 50  0001 C CNN
-F 1 "GND" H 10505 1527 50  0000 C CNN
-F 2 "" H 10500 1700 50  0001 C CNN
-F 3 "" H 10500 1700 50  0001 C CNN
-	1    10500 1700
-	1    0    0    -1
-$EndComp
-$Comp
 L Device:R R3
 U 1 1 5C0AA722
@@
 	1    0    0    -1
 $EndComp
-$Comp
-L Device:R R5
-U 1 1 5C0AA84A
-P 9700 1600
-F 0 "R5" H 9770 1646 50  0000 L CNN
-F 1 "R" H 9770 1555 50  0000 L CNN
-F 2 "Resistor_THT:R_Axial_DIN0204_L3.6mm_D1.6mm_P7.62mm_Horizontal" V 9630 1600 50  0001 C CNN
-F 3 "~" H 9700 1600 50  0001 C CNN
-	1    9700 1600
-	1    0    0    -1
-$EndComp
-$Comp
-L Device:R R6
-U 1 1 5C0AA8DC
-P 10200 1600
-F 0 "R6" H 10270 1646 50  0000 L CNN
-F 1 "R" H 10270 1555 50  0000 L CNN
-F 2 "Resistor_THT:R_Axial_DIN0204_L3.6mm_D1.6mm_P7.62mm_Horizontal" V 10130 1600 50  0001 C CNN
-F 3 "~" H 10200 1600 50  0001 C CNN
-	1    10200 1600
-	1    0    0    -1
-$EndComp
 Wire Wire Line
 	8700 1400 8700 1450
 Wire Wire Line
 	9200 1400 9200 1450
-Wire Wire Line
-	9700 1400 9700 1450
-Wire Wire Line
-	10200 1400 10200 1450
 $Comp
 L Device:R R7
@@
 $EndComp
 Wire Wire Line
-	7550 3650 7550 4000
-Wire Wire Line
 	7850 3800 8150 3800
 Wire Wire Line
 	9050 4300 9300 4300
+$Comp
+L Connector:4P4C J_joystick1
+U 1 1 5C3C1748
+P 10150 1450
+F 0 "J_joystick1" V 10159 1780 50  0000 L CNN
+F 1 "4P4C" V 10250 1780 50  0000 L CNN
+F 2 "Connector_PinHeader_2.00mm:PinHeader_1x04_P2.00mm_Vertical" V 10150 1500 50  0001 C CNN
+F 3 "~" V 10150 1500 50  0001 C CNN
+	1    10150 1450
+	0    1    1    0
+$EndComp
+$Comp
+L power:GND #PWR0111
+U 1 1 5C3C34D9
+P 10050 1850
+F 0 "#PWR0111" H 10050 1600 50  0001 C CNN
+F 1 "GND" H 10055 1677 50  0000 C CNN
+F 2 "" H 10050 1850 50  0001 C CNN
+F 3 "" H 10050 1850 50  0001 C CNN
+	1    10050 1850
+	1    0    0    -1
+$EndComp
+$Comp
+L power:VCC #PWR0112
+U 1 1 5C3C3576
+P 10350 1850
+F 0 "#PWR0112" H 10350 1700 50  0001 C CNN
+F 1 "VCC" H 10368 2023 50  0000 C CNN
+F 2 "" H 10350 1850 50  0001 C CNN
+F 3 "" H 10350 1850 50  0001 C CNN
+	1    10350 1850
+	-1   0    0    1
+$EndComp
+Text Label 10150 1950 0    50   ~ 0
+X1
+Text Label 10250 1950 0    50   ~ 0
+Y1
+Wire Wire Line
+	10150 1850 10150 1950
+Wire Wire Line
+	10250 1850 10250 1950
+$Comp
+L Connector:4P4C J_trrs1
+U 1 1 5C40CBD0
+P 7150 4100
+F 0 "J_trrs1" H 7205 4567 50  0000 C CNN
+F 1 "4P4C" H 7205 4476 50  0000 C CNN
+F 2 "Connector_PinHeader_2.00mm:PinHeader_1x04_P2.00mm_Vertical" V 7150 4150 50  0001 C CNN
+F 3 "~" V 7150 4150 50  0001 C CNN
+	1    7150 4100
+	1    0    0    -1
+$EndComp
+$Comp
+L power:VCC #PWR0101
+U 1 1 5C4148A6
+P 7550 3900
+F 0 "#PWR0101" H 7550 3750 50  0001 C CNN
+F 1 "VCC" V 7567 4028 50  0000 L CNN
+F 2 "" H 7550 3900 50  0001 C CNN
+F 3 "" H 7550 3900 50  0001 C CNN
+	1    7550 3900
+	0    1    1    0
+$EndComp
+$Comp
+L power:GND #PWR0102
+U 1 1 5C414979
+P 7550 4000
+F 0 "#PWR0102" H 7550 3750 50  0001 C CNN
+F 1 "GND" V 7555 3872 50  0000 R CNN
+F 2 "" H 7550 4000 50  0001 C CNN
+F 3 "" H 7550 4000 50  0001 C CNN
+	1    7550 4000
+	0    -1   -1   0
+$EndComp
 $EndSCHEMATC
